File: PCBs/PlateSuperior_V1/PlateSuperior_V1.kicad_pcb (KiCad board)
At the start: 2 copper layers, 116.8 x 75.8 mm, 46 parts, among them J3 Conn_02x10_Counter_Clockwise, SW1 SW_Push, SW10 SW_Push, SW11 SW_Push, SW12 SW_Push, SW13 SW_Push, SW14 SW_Push, SW15 SW_Push, SW2 SW_Push, SW3 SW_Push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

Commit message: Add top PCB
Other:
- board size 116.8 x 75.8 mm -> 106.2 x 57.3 mm
Changed lines of the file:
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@@
 	(gr_line
 		(start 126.28125 28.543934)
-		(end 126.28125 85.756066)
+		(end 126.28125 85.800018)
 		(stroke
 			(width 0.4)
@@
 	)
 	(gr_line
-		(start 26.162684 85.8)
-		(end 26.11875 85.756066)
+		(start 20.066 85.756066)
+		(end 20.066 28.5)
 		(stroke
 			(width 0.4)
@@
 	)
 	(gr_line
-		(start 26.11875 85.756066)
-		(end 26.11875 28.543934)
-		(stroke
-			(width 0.4)
-			(type default)
-		)
-		(layer "Edge.Cuts")
-	)
-	(gr_line
-		(start 26.162684 28.5)
+		(start 20.066 28.5)
 		(end 126.237316 28.5)
 		(stroke
@@
 	)
 	(gr_line
-		(start 126.237316 85.8)
-		(end 26.162684 85.8)
+		(start 126.28125 85.800018)
+		(end 20.066 85.756066)
 		(stroke
 			(width 0.4)
-			(type default)
-		)
-		(layer "Edge.Cuts")
-	)
-	(gr_line
-		(start 129.75 91)
-		(end 13.5 95.25)
-		(stroke
-			(width 0.05)
-			(type default)
-		)
-		(layer "Edge.Cuts")
-	)
-	(gr_line
-		(start 13.5 95.25)
-		(end 15 19.5)
-		(stroke
-			(width 0.05)
 			(type default)
 		)
@@
 			(type default)
 		)
-		(layer "Edge.Cuts")
-	)
-	(gr_line
-		(start 26.11875 28.543934)
-		(end 26.162684 28.5)
-		(stroke
-			(width 0.4)
-			(type default)
-		)
-		(layer "Edge.Cuts")
-	)
-	(gr_line
-		(start 130.25 20)
-		(end 129.75 91)
-		(stroke
-			(width 0.05)
-			(type default)
-		)
-		(layer "Edge.Cuts")
-	)
-	(gr_line
-		(start 126.28125 85.756066)
-		(end 126.237316 85.8)
-		(stroke
-			(width 0.4)
-			(type default)
-		)
-		(layer "Edge.Cuts")
-	)
-	(gr_line
-		(start 15 19.5)
-		(end 130.25 20)
-		(stroke
-			(width 0.05)
-			(type default)
-		)
